File: Board.sch (KiCad schematic (older format))
At the start: 5 parts, among them P1 Relay 1, P2 Relay 2, P3 Relay 3, P4 Relay 4

Commit message: Working On It
Connections:
- net labels added: 5V
- net labels removed: +12V
- no-connect marks 0 -> 1
Changed lines of the file:
@@
 LIBS:Universal
 LIBS:shield_arduino
+LIBS:Board-cache
 EELAYER 25 0
 EELAYER END
@@
 Relay4
 $Comp
-L +12V #PWR01
-U 1 1 5803B696
-P 6200 1800
-F 0 "#PWR01" H 6200 1650 50  0001 C CNN
-F 1 "+12V" H 6215 1973 50  0000 C CNN
-F 2 "" H 6200 1800 50  0000 C CNN
-F 3 "" H 6200 1800 50  0000 C CNN
-	1    6200 1800
-	1    0    0    -1
-$EndComp
-$Comp
 L ARDUINO_MEGA_SHIELD SHIELD1
 U 1 1 5803B8BE
@@
 Connection ~ 5800 1800
 $Comp
-L GND #PWR02
+L GND #PWR01
 U 1 1 5803BD43
 P 3800 4300
-F 0 "#PWR02" H 3800 4050 50  0001 C CNN
+F 0 "#PWR01" H 3800 4050 50  0001 C CNN
 F 1 "GND" H 3805 4127 50  0000 C CNN
 F 2 "" H 3800 4300 50  0000 C CNN
@@
 	-1   0    0    1
 $EndComp
+$Comp
+L GND #PWR?
+U 1 1 5803ED68
+P 3900 4300
+F 0 "#PWR?" H 3900 4050 50  0001 C CNN
+F 1 "GND" H 3905 4127 50  0000 C CNN
+F 2 "" H 3900 4300 50  0000 C CNN
+F 3 "" H 3900 4300 50  0000 C CNN
+	1    3900 4300
+	-1   0    0    1
+$EndComp
+$Comp
+L GND #PWR?
+U 1 1 5803ED82
+P 6050 4300
+F 0 "#PWR?" H 6050 4050 50  0001 C CNN
+F 1 "GND" H 6055 4127 50  0000 C CNN
+F 2 "" H 6050 4300 50  0000 C CNN
+F 3 "" H 6050 4300 50  0000 C CNN
+	1    6050 4300
+	-1   0    0    1
+$EndComp
+$Comp
+L GND #PWR?
+U 1 1 5803ED9C
+P 6150 4300
+F 0 "#PWR?" H 6150 4050 50  0001 C CNN
+F 1 "GND" H 6155 4127 50  0000 C CNN
+F 2 "" H 6150 4300 50  0000 C CNN
+F 3 "" H 6150 4300 50  0000 C CNN
+	1    6150 4300
+	-1   0    0    1
+$EndComp
+$Comp
+L GND #PWR?
+U 1 1 5803EDB6
+P 6750 6200
+F 0 "#PWR?" H 6750 5950 50  0001 C CNN
+F 1 "GND" H 6755 6027 50  0000 C CNN
+F 2 "" H 6750 6200 50  0000 C CNN
+F 3 "" H 6750 6200 50  0000 C CNN
+	1    6750 6200
+	1    0    0    -1
+$EndComp
+$Comp
+L GND #PWR?
+U 1 1 5803EE20
+P 7250 6200
+F 0 "#PWR?" H 7250 5950 50  0001 C CNN
+F 1 "GND" H 7255 6027 50  0000 C CNN
+F 2 "" H 7250 6200 50  0000 C CNN
+F 3 "" H 7250 6200 50  0000 C CNN
+	1    7250 6200
+	1    0    0    -1
+$EndComp
+Text GLabel 4000 6200 3    60   BiDi ~ 0
+5V
+Text GLabel 4100 6200 3    60   BiDi ~ 0
+5V
+Text GLabel 6250 4300 1    60   BiDi ~ 0
+5V
+Text GLabel 6200 1800 2    60   BiDi ~ 0
+5V
+NoConn ~ 6650 4300
 $EndSCHEMATC

Commit message: Pins are in
Parts:
- added P10, P11: CONN_01X18, Pin_Headers:Pin_Header_Straight_1x18, symbol CONN_01X18
- added P12: CONN_01X06, Pin_Headers:Pin_Header_Straight_1x06, symbol CONN_01X06
- added P5, P6, P7, P8, P9: CONN_01X08, Pin_Headers:Pin_Header_Straight_1x08, symbol CONN_01X08
Connections:
- net 5V: now also P10.1 (P1), P11.1 (P1), P12.3 (P3)
- net GND: now also P10.18 (P18), P11.18 (P18), P12.4 (P4), P12.5 (P5), P5.2 (P2)
- net Relay1: now also P10.16 (P16)
- net Relay2: now also P11.16 (P16)
- net Relay3: now also P10.17 (P17)
- net Relay4: now also P11.17 (P17)
- net RX: now reaches SHIELD1.0 (RX0)
- net RX: now also P6.8 (P8)
- net TX: now reaches SHIELD1.1 (TX0)
- net TX: now also P6.7 (P7)
- net 10: now reaches SHIELD1.10
- net 10: now also P5.6 (P6)
- net 11: now reaches SHIELD1.11
- net 11: now also P5.5 (P5)
- net 12: now reaches SHIELD1.12
- net 12: now also P5.4 (P4)
- net 13: now reaches SHIELD1.13
- net 13: now also P5.3 (P3)
- net TX3: now reaches SHIELD1.14 (TX3)
- net TX3: now also P7.1 (P1)
- net RX3: now reaches SHIELD1.15 (RX3)
- net RX3: now also P7.2 (P2)
- net TX2: now reaches SHIELD1.16 (TX2)
- net TX2: now also P7.3 (P3)
- net RX2: now reaches SHIELD1.17 (RX2)
- net RX2: now also P7.4 (P4)
- net TX1: now reaches SHIELD1.18 (TX1)
- net TX1: now also P7.5 (P5)
- net RX1: now reaches SHIELD1.19 (RX1)
- net RX1: now also P7.6 (P6)
- net 2: now reaches SHIELD1.2
- net 2: now also P6.6 (P6)
- net SDA: now reaches SHIELD1.20 (SDA)
- net SDA: now also P7.7 (P7)
- net SCL: now reaches SHIELD1.21 (SCL)
- net SCL: now also P7.8 (P8)
- net PA0: now reaches SHIELD1.22 (PA0)
- net PA0: now also P10.2 (P2)
- net PA1: now reaches SHIELD1.23 (PA1)
- net PA1: now also P11.2 (P2)
- net PA2: now reaches SHIELD1.24 (PA2)
- net PA2: now also P10.3 (P3)
- net PA3: now reaches SHIELD1.25 (PA3)
- net PA3: now also P11.3 (P3)
- net PA4: now reaches SHIELD1.26 (PA4)
- net PA4: now also P10.4 (P4)
- net PA5: now reaches SHIELD1.27 (PA5)
- net PA5: now also P11.4 (P4)
- net PA6: now reaches SHIELD1.28 (PA6)
- net PA6: now also P10.5 (P5)
- net PA7: now reaches SHIELD1.29 (PA7)
- net PA7: now also P11.5 (P5)
- net 3: now reaches SHIELD1.3
- net 3: now also P6.5 (P5)
- net PC7: now reaches SHIELD1.30 (PC7)
- net PC7: now also P10.6 (P6)
- net PC6: now reaches SHIELD1.31 (PC6)
- net PC6: now also P11.6 (P6)
- net PC5: now reaches SHIELD1.32 (PC5)
- net PC5: now also P10.7 (P7)
- net PC4: now reaches SHIELD1.33 (PC4)
- net PC4: now also P11.7 (P7)
- net PC3: now reaches SHIELD1.34 (PC3)
- net PC3: now also P10.8 (P8)
- net PC2: now reaches SHIELD1.35 (PC2)
- net PC2: now also P11.8 (P8)
- net PC1: now reaches SHIELD1.36 (PC1)
- net PC1: now also P10.9 (P9)
- net PC0: now reaches SHIELD1.37 (PC0)
- net PC0: now also P11.9 (P9)
- net PD7: now reaches SHIELD1.38 (PD7)
- net PD7: now also P10.10 (P10)
- net PG2: now reaches SHIELD1.39 (PG2)
- net PG2: now also P11.10 (P10)
- net 3V: now reaches SHIELD1.3V3
- net 3V: now also P12.2 (P2)
- net 4: now reaches SHIELD1.4
- net 4: now also P6.4 (P4)
- net PG1: now reaches SHIELD1.40 (PG1)
- net PG1: now also P10.11 (P11)
- net PG0: now reaches SHIELD1.41 (PG0)
- net PG0: now also P11.11 (P11)
- net PL7: now reaches SHIELD1.42 (PL7)
- net PL7: now also P10.12 (P12)
- net PL6: now reaches SHIELD1.43 (PL6)
- net PL6: now also P11.12 (P12)
- net PL5: now reaches SHIELD1.44 (PL5)
- net PL5: now also P10.13 (P13)
- net PL4: now reaches SHIELD1.45 (PL4)
- net PL4: now also P11.13 (P13)
- net PL3: now reaches SHIELD1.46 (PL3)
- net PL3: now also P10.14 (P14)
- net PL2: now reaches SHIELD1.47 (PL2)
- net PL2: now also P11.14 (P14)
- net PL1: now reaches SHIELD1.48 (PL1)
- net PL1: now also P10.15 (P15)
- net PL0: now reaches SHIELD1.49 (PL0)
- net PL0: now also P11.15 (P15)
- net 5: now reaches SHIELD1.5
- net 5: now also P6.3 (P3)
- net 6: now reaches SHIELD1.6
- net 6: now also P6.2 (P2)
- net 7: now reaches SHIELD1.7
- net 7: now also P6.1 (P1)
- net 8: now reaches SHIELD1.8
- net 8: now also P5.8 (P8)
- net 9: now reaches SHIELD1.9
- net 9: now also P5.7 (P7)
- net AD0: now reaches SHIELD1.AD0
- net AD0: now also P8.1 (P1)
- net AD1: now reaches SHIELD1.AD1
- net AD1: now also P8.2 (P2)
- net AD10: now reaches SHIELD1.AD10
- net AD10: now also P9.3 (P3)
- net AD11: now reaches SHIELD1.AD11
- net AD11: now also P9.4 (P4)
- net AD12: now reaches SHIELD1.AD12
- net AD12: now also P9.5 (P5)
- net AD13: now reaches SHIELD1.AD13
- net AD13: now also P9.6 (P6)
- net AD14: now reaches SHIELD1.AD14
- net AD14: now also P9.7 (P7)
- net AD15: now reaches SHIELD1.AD15
- net AD15: now also P9.8 (P8)
- net AD2: now reaches SHIELD1.AD2
- net AD2: now also P8.3 (P3)
- net AD3: now reaches SHIELD1.AD3
- net AD3: now also P8.4 (P4)
- net AD4: now reaches SHIELD1.AD4
- net AD4: now also P8.5 (P5)
- net AD5: now reaches SHIELD1.AD5
- net AD5: now also P8.6 (P6)
- net AD6: now reaches SHIELD1.AD6
- net AD6: now also P8.7 (P7)
- net AD7: now reaches SHIELD1.AD7
- net AD7: now also P8.8 (P8)
- net AD8: now reaches SHIELD1.AD8
- net AD8: now also P9.1 (P1)
- net AD9: now reaches SHIELD1.AD9
- net AD9: now also P9.2 (P2)
- net AREF: now reaches SHIELD1.AREF
- net AREF: now also P5.1 (P1)
- net RST: now reaches SHIELD1.RST
- net RST: now also P12.1 (P1)
- net V_IN: now reaches SHIELD1.V_IN
- net V_IN: now also P12.6 (P6)
- no-connect marks 1 -> 9
Other:
- moved on the sheet: P1, P2, P3, P4

Commit message: Working on Relays
Parts:
- added RLY1, RLY2, RLY3, RLY4: RELAY_40.31, Relays_THT:Relay_SPDS_OMRON-G6E, symbol RELAY_40.31
Changed lines of the file:
@@
 NoConn ~ 7050 6200
 NoConn ~ 6950 6200
+$Comp
+L RELAY_40.31 RLY1
+U 1 1 5807B24D
+P 7900 3500
+F 0 "RLY1" H 7900 3897 60  0000 C CNN
+F 1 "RELAY_40.31" H 7900 3791 60  0000 C CNN
+F 2 "Relays_THT:Relay_SPDS_OMRON-G6E" H 7900 3500 60  0001 C CNN
+F 3 "http://www.mouser.com/ds/2/307/G6E_0911-7980.pdf" H 7900 3500 60  0001 C CNN
+F 4 "G6E-134P-US DC5" H 7900 3500 60  0001 C CNN "manf#"
+	1    7900 3500
+	1    0    0    -1
+$EndComp
+$Comp
+L RELAY_40.31 RLY2
+U 1 1 5807B29F
+P 8650 3500
+F 0 "RLY2" H 8650 3897 60  0000 C CNN
+F 1 "RELAY_40.31" H 8650 3791 60  0000 C CNN
+F 2 "Relays_THT:Relay_SPDS_OMRON-G6E" H 8650 3500 60  0001 C CNN
+F 3 "" H 8650 3500 60  0000 C CNN
+	1    8650 3500
+	1    0    0    -1
+$EndComp
+$Comp
+L RELAY_40.31 RLY3
+U 1 1 5807B2FA
+P 9400 3500
+F 0 "RLY3" H 9400 3897 60  0000 C CNN
+F 1 "RELAY_40.31" H 9400 3791 60  0000 C CNN
+F 2 "Relays_THT:Relay_SPDS_OMRON-G6E" H 9400 3500 60  0001 C CNN
+F 3 "" H 9400 3500 60  0000 C CNN
+	1    9400 3500
+	1    0    0    -1
+$EndComp
+$Comp
+L RELAY_40.31 RLY4
+U 1 1 5807B34E
+P 10050 3500
+F 0 "RLY4" H 10050 3897 60  0000 C CNN
+F 1 "RELAY_40.31" H 10050 3791 60  0000 C CNN
+F 2 "Relays_THT:Relay_SPDS_OMRON-G6E" H 10050 3500 60  0001 C CNN
+F 3 "" H 10050 3500 60  0000 C CNN
+	1    10050 3500
+	1    0    0    -1
+$EndComp
 $EndSCHEMATC

Commit message: Cleaning Up Board
Parts:
- added D1, D3, D5, D6: RED, LEDs:LED-3MM, symbol LED
- added D2, D4, D7, D8: 1N4148, Diodes_ThroughHole:Diode_DO-35_SOD27_Horizontal_RM10, symbol D
- added Q1, Q2, Q3, Q4: PN2222A, TO_SOT_Packages_THT:TO-92_Inline_Narrow_Oval, symbol PN2222A
- added R1, R4, R7, R8: 470, Resistors_ThroughHole:Resistor_Horizontal_RM7mm, symbol R
- added R2, R3, R5, R6: 2.2K, Resistors_ThroughHole:Resistor_Horizontal_RM7mm, symbol R
- P3: value Relay 3 -> Relay 4
- P4: value Relay 4 -> Relay 3
- RLY1: footprint Relays_THT:Relay_SPDS_OMRON-G6E -> Relays_ThroughHole:Relay_SPDS_OMRON-G6E
- RLY2, RLY3, RLY4: footprint Relays_THT:Relay_SPDS_OMRON-G6E -> Relays_ThroughHole:Relay_SPDS_OMRON-G6E; manf# (none) -> G6E-134P-US DC5
- SHIELD1: manf# (none) -> 2893
Connections:
- net 10: no longer SHIELD1.10
- net 11: no longer SHIELD1.11
- net 12: no longer SHIELD1.12
- net 13: no longer SHIELD1.13
- net 2: no longer SHIELD1.2
- net 3: no longer SHIELD1.3
- net 3V: no longer SHIELD1.3V3
- net 4: no longer SHIELD1.4
- net 5: no longer SHIELD1.5
- net 5V: no longer P1.2 (P2), P2.2 (P2), P3.2 (P2), P4.2 (P2), SHIELD1.5V, SHIELD1.5V_4, SHIELD1.5V_5
- net 6: no longer SHIELD1.6
- net 7: no longer SHIELD1.7
- net 8: no longer SHIELD1.8
- net 9: no longer SHIELD1.9
- net AD0: no longer SHIELD1.AD0
- net AD1: no longer SHIELD1.AD1
- net AD10: no longer SHIELD1.AD10
- net AD11: no longer SHIELD1.AD11
- net AD12: no longer SHIELD1.AD12
- net AD13: no longer SHIELD1.AD13
- net AD14: no longer SHIELD1.AD14
- net AD15: no longer SHIELD1.AD15
- net AD2: no longer SHIELD1.AD2
- net AD3: no longer SHIELD1.AD3
- net AD4: no longer SHIELD1.AD4
- net AD5: no longer SHIELD1.AD5
- net AD6: no longer SHIELD1.AD6
- net AD7: no longer SHIELD1.AD7
- net AD8: no longer SHIELD1.AD8
- net AD9: no longer SHIELD1.AD9
- net AREF: no longer SHIELD1.AREF
- net GND: now also Q1.1 (E), Q2.1 (E), Q3.1 (E), Q4.1 (E); no longer SHIELD1.GND1, SHIELD1.GND2, SHIELD1.GND3, SHIELD1.GND4, SHIELD1.GND5
- net PA0: no longer SHIELD1.22 (PA0)
- net PA1: no longer SHIELD1.23 (PA1)
- net PA2: no longer SHIELD1.24 (PA2)
- net PA3: no longer SHIELD1.25 (PA3)
- net PA4: no longer SHIELD1.26 (PA4)
- net PA5: no longer SHIELD1.27 (PA5)
- net PA6: no longer SHIELD1.28 (PA6)
- net PA7: no longer SHIELD1.29 (PA7)
- net PC0: no longer SHIELD1.37 (PC0)
- net PC1: no longer SHIELD1.36 (PC1)
- net PC2: no longer SHIELD1.35 (PC2)
- net PC3: no longer SHIELD1.34 (PC3)
- net PC4: no longer SHIELD1.33 (PC4)
- net PC5: no longer SHIELD1.32 (PC5)
- net PC6: no longer SHIELD1.31 (PC6)
- net PC7: no longer SHIELD1.30 (PC7)
- net PD7: no longer SHIELD1.38 (PD7)
- net PG0: no longer SHIELD1.41 (PG0)
- net PG1: no longer SHIELD1.40 (PG1)
- net PG2: no longer SHIELD1.39 (PG2)
- net PL0: no longer SHIELD1.49 (PL0)
- net PL1: no longer SHIELD1.48 (PL1)
- net PL2: no longer SHIELD1.47 (PL2)
- net PL3: no longer SHIELD1.46 (PL3)
- net PL4: no longer SHIELD1.45 (PL4)
- net PL5: no longer SHIELD1.44 (PL5)
- net PL6: no longer SHIELD1.43 (PL6)
- net PL7: no longer SHIELD1.42 (PL7)
- net RST: no longer SHIELD1.RST
- net RX: no longer SHIELD1.0 (RX0)
- net RX1: no longer SHIELD1.19 (RX1)
- net RX2: no longer SHIELD1.17 (RX2)
- net RX3: no longer SHIELD1.15 (RX3)
- net Relay1: now also P10.17 (P17), R2.2; no longer P1.1 (P1), P10.16 (P16), SHIELD1.50 (PB3_(MISO))
- net Relay2: now also P11.17 (P17), R3.2; no longer P11.16 (P16), P2.1 (P1), SHIELD1.51 (PB2_(MOSI))
- net Relay3: now also P10.16 (P16), R5.2; no longer P10.17 (P17), P3.1 (P1), SHIELD1.52 (PB1_(SCK))
- net Relay4: now also P11.16 (P16), R6.2; no longer P11.17 (P17), P4.1 (P1), SHIELD1.53 (PB0_(SS))
- net SCL: no longer SHIELD1.21 (SCL)
- net SDA: no longer SHIELD1.20 (SDA)
- net TX: no longer SHIELD1.1 (TX0)
- net TX1: no longer SHIELD1.18 (TX1)
- net TX2: no longer SHIELD1.16 (TX2)
- net TX3: no longer SHIELD1.14 (TX3)
- net V_IN: no longer SHIELD1.V_IN
- net at RLY1.1: now also D2.2 (A), Q1.3 (C), R1.2
- net at RLY1.12: now also P1.1 (P1)
- net at RLY1.6: now also D1.2 (A), D2.1 (K)
- net at RLY1.7: now also P1.2 (P2)
- net at RLY2.1: now also D4.2 (A), Q2.3 (C), R4.2
- net at RLY2.12: now also P2.1 (P1)
- net at RLY2.6: now also D3.2 (A), D4.1 (K)
- net at RLY2.7: now also P2.2 (P2)
- net at RLY3.1: now also D7.2 (A), Q3.3 (C), R7.2
- net at RLY3.12: now also P3.1 (P1)
- net at RLY3.6: now also D5.2 (A), D7.1 (K)
- net at RLY3.7: now also P3.2 (P2)
- net at RLY4.1: now also D8.2 (A), Q4.3 (C), R8.2
- net at RLY4.12: now also P4.1 (P1)
- net at RLY4.6: now also D6.2 (A), D8.1 (K)
- net at RLY4.7: now also P4.2 (P2)
- new net: D1.1 (K), R1.1
- new net: Q1.2 (B), R2.1
- new net: D3.1 (K), R4.1
- new net: Q2.2 (B), R3.1
- new net: D6.1 (K), R8.1
- new net: Q4.2 (B), R6.1
- new net: D5.1 (K), R7.1
- new net: Q3.2 (B), R5.1
- no-connect marks 9 -> 95
Other:
- moved on the sheet: P1, RLY1, SHIELD1

Commit message: Finishing up board
Connections:
- net 5V: no longer P10.1 (P1), P11.1 (P1)
- no-connect marks 95 -> 97
Changed lines of the file:
@@
 Text GLabel 7400 950  0    60   BiDi ~ 0
 PA1
-Text GLabel 7400 850  0    60   BiDi ~ 0
-5V
-Text GLabel 8500 850  0    60   BiDi ~ 0
-5V
 Text GLabel 8500 2250 0    60   BiDi ~ 0
 PL1
@@
 Text GLabel 8500 2450 0    60   BiDi ~ 0
 Relay1
+NoConn ~ 8500 850
+NoConn ~ 7400 850
 $EndSCHEMATC
